File: Input_Output_Buffers.kicad_sch (KiCad schematic)
At the start: 35 parts, among them J1 Conn_02x07_Odd_Even, J4 Conn_02x07_Odd_Even, U1 74HC245, U2 74HC245, U26 74HC245, U27 74HC245

Commit message: sample
Changed lines of the file:
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@@
 	)
 	(junction
+		(at 45.72 74.93)
+		(diameter 0)
+		(color 0 0 0 0)
+	)
+	(junction
 		(at 184.15 92.71)
 		(diameter 0)
@@
 	)
 	(junction
+		(at 58.42 88.9)
+		(diameter 0)
+		(color 0 0 0 0)
+	)
+	(junction
 		(at 180.34 20.32)
 		(diameter 0)
@@
 	)
 	(junction
-		(at 207.01 16.51)
-		(diameter 0)
-		(color 0 0 0 0)
-	)
-	(junction
 		(at 199.39 92.71)
 		(diameter 0)
@@
 	)
 	(junction
-		(at 58.42 88.9)
-		(diameter 0)
-		(color 0 0 0 0)
-	)
-	(junction
 		(at 85.09 102.87)
 		(diameter 0)
@@
 	)
 	(junction
-		(at 45.72 77.47)
-		(diameter 0)
-		(color 0 0 0 0)
-	)
-	(junction
 		(at 31.75 147.32)
 		(diameter 0)
@@
 	(wire
 		(pts
-			(xy 45.72 72.39) (xy 38.1 72.39)
-		)
-		(stroke
-			(width 0)
-			(type default)
-		)
-	)
-	(wire
-		(pts
 			(xy 154.94 102.87) (xy 154.94 111.76)
 		)
@@
 	(wire
 		(pts
-			(xy 38.1 77.47) (xy 45.72 77.47)
+			(xy 257.81 156.21) (xy 267.97 156.21)
 		)
 		(stroke
@@
 	(wire
 		(pts
-			(xy 257.81 156.21) (xy 267.97 156.21)
+			(xy 215.9 66.04) (xy 167.64 66.04)
 		)
 		(stroke
@@
 	(wire
 		(pts
-			(xy 215.9 66.04) (xy 167.64 66.04)
+			(xy 85.09 115.57) (xy 85.09 134.62)
 		)
 		(stroke
@@
 	(wire
 		(pts
-			(xy 85.09 115.57) (xy 85.09 134.62)
+			(xy 35.56 54.61) (xy 45.72 54.61)
 		)
 		(stroke
@@
 	(wire
 		(pts
-			(xy 35.56 54.61) (xy 45.72 54.61)
+			(xy 184.15 92.71) (xy 191.77 92.71)
 		)
 		(stroke
@@
 	(wire
 		(pts
-			(xy 184.15 92.71) (xy 191.77 92.71)
+			(xy 137.16 132.08) (xy 142.24 132.08)
 		)
 		(stroke
@@
 	(wire
 		(pts
-			(xy 45.72 77.47) (xy 45.72 88.9)
+			(xy 45.72 74.93) (xy 45.72 88.9)
 		)
 		(stroke
@@
 	(wire
 		(pts
-			(xy 38.1 72.39) (xy 38.1 77.47)
+			(xy 45.72 72.39) (xy 45.72 74.93)
 		)
 		(stroke
@@
 	(wire
 		(pts
-			(xy 45.72 74.93) (xy 45.72 77.47)
-		)
-		(stroke
-			(width 0)
-			(type default)
-		)
-	)
-	(wire
-		(pts
 			(xy 205.74 129.54) (xy 167.64 129.54)
 		)
@@
 	(wire
 		(pts
-			(xy 133.35 129.54) (xy 142.24 129.54)
-		)
-		(stroke
-			(width 0)
-			(type default)
-		)
-	)
-	(wire
-		(pts
 			(xy 167.64 137.16) (xy 226.06 137.16)
 		)
@@
 	(wire
 		(pts
+			(xy 128.27 134.62) (xy 142.24 134.62)
+		)
+		(stroke
+			(width 0)
+			(type default)
+		)
+	)
+	(wire
+		(pts
 			(xy 33.02 139.7) (xy 43.18 139.7)
 		)
@@
 	(wire
 		(pts
-			(xy 207.01 15.24) (xy 207.01 16.51)
-		)
-		(stroke
-			(width 0)
-			(type default)
-		)
-	)
-	(wire
-		(pts
 			(xy 203.2 20.32) (xy 209.55 20.32)
 		)
@@
 	(wire
 		(pts
-			(xy 196.85 58.42) (xy 220.98 58.42)
+			(xy 137.16 137.16) (xy 142.24 137.16)
 		)
 		(stroke
@@
 	(wire
 		(pts
-			(xy 209.55 92.71) (xy 213.36 92.71)
+			(xy 196.85 58.42) (xy 220.98 58.42)
 		)
 		(stroke
@@
 	(wire
 		(pts
-			(xy 203.2 60.96) (xy 167.64 60.96)
+			(xy 209.55 92.71) (xy 213.36 92.71)
 		)
 		(stroke
@@
 	(wire
 		(pts
-			(xy 243.84 82.55) (xy 251.46 82.55)
+			(xy 203.2 60.96) (xy 167.64 60.96)
 		)
 		(stroke
@@
 	(wire
 		(pts
-			(xy 68.58 129.54) (xy 77.47 129.54)
+			(xy 243.84 82.55) (xy 251.46 82.55)
 		)
 		(stroke
@@
 	(wire
 		(pts
-			(xy 190.5 40.64) (xy 190.5 55.88)
+			(xy 68.58 129.54) (xy 77.47 129.54)
 		)
 		(stroke
@@
 	(wire
 		(pts
-			(xy 133.35 137.16) (xy 142.24 137.16)
+			(xy 190.5 40.64) (xy 190.5 55.88)
 		)
 		(stroke
@@
 	(wire
 		(pts
-			(xy 133.35 132.08) (xy 142.24 132.08)
+			(xy 78.74 49.53) (xy 71.12 49.53)
 		)
 		(stroke
@@
 	(wire
 		(pts
-			(xy 78.74 49.53) (xy 71.12 49.53)
+			(xy 34.29 129.54) (xy 43.18 129.54)
 		)
 		(stroke
@@
 	(wire
 		(pts
-			(xy 34.29 129.54) (xy 43.18 129.54)
+			(xy 245.11 161.29) (xy 227.33 161.29)
 		)
 		(stroke
@@
 	(wire
 		(pts
-			(xy 245.11 161.29) (xy 227.33 161.29)
+			(xy 91.44 20.32) (xy 97.79 20.32)
 		)
 		(stroke
@@
 	(wire
 		(pts
-			(xy 91.44 20.32) (xy 97.79 20.32)
+			(xy 243.84 80.01) (xy 251.46 80.01)
 		)
 		(stroke
@@
 	(wire
 		(pts
-			(xy 243.84 80.01) (xy 251.46 80.01)
+			(xy 138.43 144.78) (xy 138.43 152.4)
 		)
 		(stroke
@@
 	(wire
 		(pts
-			(xy 138.43 144.78) (xy 138.43 152.4)
+			(xy 196.85 20.32) (xy 203.2 20.32)
 		)
 		(stroke
@@
 	(wire
 		(pts
-			(xy 196.85 20.32) (xy 203.2 20.32)
+			(xy 63.5 88.9) (xy 58.42 88.9)
 		)
 		(stroke
@@
 	(wire
 		(pts
-			(xy 133.35 134.62) (xy 142.24 134.62)
-		)
-		(stroke
-			(width 0)
-			(type default)
-		)
-	)
-	(wire
-		(pts
 			(xy 43.18 154.94) (xy 43.18 168.91)
 		)
@@
 	(wire
 		(pts
+			(xy 128.27 129.54) (xy 142.24 129.54)
+		)
+		(stroke
+			(width 0)
+			(type default)
+		)
+	)
+	(wire
+		(pts
 			(xy 190.5 55.88) (xy 167.64 55.88)
 		)
@@
 	(global_label "DATA_OUT4"
 		(shape input)
-		(at 133.35 137.16 180)
+		(at 137.16 137.16 180)
 		(fields_autoplaced yes)
 		(effects
@@
 		)
 		(property "Intersheetrefs" "${INTERSHEET_REFS}"
-			(at 120.1443 137.16 0)
+			(at 123.9543 137.16 0)
 			(hide yes)
 			(show_name no)
@@
 	(global_label "DATA_OUT3"
 		(shape input)
-		(at 133.35 134.62 180)
+		(at 128.27 134.62 180)
 		(fields_autoplaced yes)
 		(effects
@@
 		)
 		(property "Intersheetrefs" "${INTERSHEET_REFS}"
-			(at 120.1443 134.62 0)
+			(at 115.0643 134.62 0)
 			(hide yes)
 			(show_name no)
@@
 	(global_label "DATA_OUT2"
 		(shape input)
-		(at 133.35 132.08 180)
+		(at 137.16 132.08 180)
 		(fields_autoplaced yes)
 		(effects
@@
 		)
 		(property "Intersheetrefs" "${INTERSHEET_REFS}"
-			(at 120.1443 132.08 0)
+			(at 123.9543 132.08 0)
 			(hide yes)
 			(show_name no)
@@
 	(global_label "DATA_OUT1"
 		(shape input)
-		(at 133.35 129.54 180)
+		(at 128.27 129.54 180)
 		(fields_autoplaced yes)
 		(effects
@@
 		)
 		(property "Intersheetrefs" "${INTERSHEET_REFS}"
-			(at 120.1443 129.54 0)
+			(at 115.0643 129.54 0)
 			(hide yes)
 			(show_name no)
@@
 	(symbol
 		(lib_id "power:GND")
-		(at 58.42 88.9 0)
+		(at 63.5 88.9 0)
 		(unit 1)
 		(body_style 1)
@@
 		(fields_autoplaced yes)
 		(property "Reference" "#PWR019"
-			(at 58.42 95.25 0)
+			(at 63.5 95.25 0)
 			(hide yes)
 			(show_name no)
@@
 		)
 		(property "Value" "GND"
-			(at 58.42 93.98 0)
+			(at 63.5 93.98 0)
 			(show_name no)
 			(do_not_autoplace no)
@@
 		)
 		(property "Footprint" ""
-			(at 58.42 88.9 0)
+			(at 63.5 88.9 0)
 			(hide yes)
 			(show_name no)
@@
 		)
 		(property "Datasheet" ""
-			(at 58.42 88.9 0)
+			(at 63.5 88.9 0)
 			(hide yes)
 			(show_name no)
@@
 		)
 		(property "Description" "Power symbol creates a global label with name \"GND\" , ground"
-			(at 58.42 88.9 0)
+			(at 63.5 88.9 0)
 			(hide yes)
 			(show_name no)

Commit message: Updated PCB
Parts:
- removed DC90, DC91: 0.1uF, Capacitor_SMD:C_0805_2012Metric, symbol Device:C
- removed R216, R217, R220, R221, R222, R223, R224, R225, R226, R227, R228: 4.7K, Resistor_SMD:R_0805_2012Metric, symbol Device:R
- removed U26, U27: 74HC245, Package_SO:TSSOP-20_4.4x6.5mm_P0.65mm, symbol 74xx:74HC245
- U1, U2: footprint Package_SO:TSSOP-20_4.4x6.5mm_P0.65mm -> (none)
Connections:
- net B2_LATCH is gone; now on net LATCH_OUT: R2.2, U1.17 (B1)
- net B2_OE is gone; now on net OE_OUT: R213.2, U1.15 (B3)
- net B2_SCLK is gone; now on net SCLK_OUT: R214.2, U1.13 (B5)
- net DATA_1_OUT is gone; now on net DATA_OUT1: J1.7 (Pin_7)
- net DATA_2_OUT is gone; now on net DATA_OUT2: J1.8 (Pin_8)
- net DATA_3_OUT is gone; now on net DATA_OUT3: J1.9 (Pin_9)
- net DATA_4_OUT is gone; now on net DATA_OUT4: J1.10 (Pin_10)
- net ROWA_OUT is gone; now on net ROWA: J1.3 (Pin_3)
- net ROWB_OUT is gone; now on net ROWB: J1.4 (Pin_4)
- net ROWC_OUT is gone; now on net ROWC: J1.5 (Pin_5)
- net ROWD_OUT is gone; now on net ROWD: J1.6 (Pin_6)
- no-connect marks 14 -> 6
Other:
- moved on the sheet: DC1, DC2, J1, J4, R1, R10, R11, R2, R213, R214, R215, R3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
