File: LED_DRIVER.kicad_sch (KiCad schematic)
At the start: 22 parts

Commit message: Updated PCB
Changed lines of the file:
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@@
-	)
-	(junction
-		(at 113.03 69.85)
-		(diameter 0)
-		(color 0 0 0 0)
-	)
-	(junction
-		(at 241.3 63.5)
-		(diameter 0)
-		(color 0 0 0 0)
 	)
 	(junction
@@
 	)
 	(junction
-		(at 113.03 64.77)
-		(diameter 0)
-		(color 0 0 0 0)
-	)
-	(junction
 		(at 102.87 64.77)
 		(diameter 0)
@@
 	)
 	(junction
-		(at 241.3 68.58)
-		(diameter 0)
-		(color 0 0 0 0)
-	)
-	(junction
 		(at 201.93 35.56)
 		(diameter 0)
@@
 	(wire
 		(pts
-			(xy 241.3 71.12) (xy 248.92 71.12)
-		)
-		(stroke
-			(width 0)
-			(type default)
-		)
-	)
-	(wire
-		(pts
 			(xy 88.9 36.83) (xy 88.9 41.91)
 		)
@@
 	(wire
 		(pts
-			(xy 113.03 67.31) (xy 120.65 67.31)
-		)
-		(stroke
-			(width 0)
-			(type default)
-		)
-	)
-	(wire
-		(pts
-			(xy 113.03 64.77) (xy 113.03 67.31)
-		)
-		(stroke
-			(width 0)
-			(type default)
-		)
-	)
-	(wire
-		(pts
 			(xy 46.99 64.77) (xy 46.99 63.5)
 		)
@@
 	(wire
 		(pts
-			(xy 113.03 72.39) (xy 120.65 72.39)
-		)
-		(stroke
-			(width 0)
-			(type default)
-		)
-	)
-	(wire
-		(pts
 			(xy 55.88 55.88) (xy 55.88 50.8)
 		)
@@
 	(wire
 		(pts
-			(xy 241.3 68.58) (xy 241.3 71.12)
-		)
-		(stroke
-			(width 0)
-			(type default)
-		)
-	)
-	(wire
-		(pts
 			(xy 73.66 50.8) (xy 73.66 48.26)
 		)
@@
 	(wire
 		(pts
-			(xy 113.03 69.85) (xy 128.27 69.85)
-		)
-		(stroke
-			(width 0)
-			(type default)
-		)
-	)
-	(wire
-		(pts
 			(xy 175.26 49.53) (xy 184.15 49.53)
 		)
@@
 	(wire
 		(pts
-			(xy 113.03 69.85) (xy 113.03 72.39)
-		)
-		(stroke
-			(width 0)
-			(type default)
-		)
-	)
-	(wire
-		(pts
 			(xy 67.31 64.77) (xy 46.99 64.77)
 		)
@@
 	(wire
 		(pts
-			(xy 104.14 69.85) (xy 113.03 69.85)
-		)
-		(stroke
-			(width 0)
-			(type default)
-		)
-	)
-	(wire
-		(pts
-			(xy 102.87 64.77) (xy 113.03 64.77)
+			(xy 104.14 69.85) (xy 128.27 69.85)
+		)
+		(stroke
+			(width 0)
+			(type default)
+		)
+	)
+	(wire
+		(pts
+			(xy 102.87 64.77) (xy 127 64.77)
 		)
 		(stroke
@@
 	(wire
 		(pts
-			(xy 241.3 63.5) (xy 241.3 66.04)
-		)
-		(stroke
-			(width 0)
-			(type default)
-		)
-	)
-	(wire
-		(pts
 			(xy 201.93 46.99) (xy 209.55 46.99)
 		)
@@
 	(wire
 		(pts
-			(xy 241.3 66.04) (xy 248.92 66.04)
-		)
-		(stroke
-			(width 0)
-			(type default)
-		)
-	)
-	(wire
-		(pts
 			(xy 175.26 63.5) (xy 175.26 62.23)
 		)
@@
 	(wire
 		(pts
-			(xy 232.41 68.58) (xy 241.3 68.58)
+			(xy 232.41 68.58) (xy 257.81 68.58)
 		)
 		(stroke
@@
 	(wire
 		(pts
-			(xy 241.3 63.5) (xy 257.81 63.5)
+			(xy 232.41 63.5) (xy 257.81 63.5)
 		)
 		(stroke
@@
 	(wire
 		(pts
-			(xy 241.3 68.58) (xy 257.81 68.58)
-		)
-		(stroke
-			(width 0)
-			(type default)
-		)
-	)
-	(wire
-		(pts
-			(xy 113.03 64.77) (xy 127 64.77)
-		)
-		(stroke
-			(width 0)
-			(type default)
-		)
-	)
-	(wire
-		(pts
 			(xy 232.41 49.53) (xy 232.41 54.61)
 		)
@@
 		(pts
 			(xy 161.29 66.04) (xy 175.26 66.04)
-		)
-		(stroke
-			(width 0)
-			(type default)
-		)
-	)
-	(wire
-		(pts
-			(xy 232.41 63.5) (xy 241.3 63.5)
 		)
 		(stroke
@@
 		)
 	)
-	(global_label "TR32"
-		(shape input)
-		(at 248.92 66.04 0)
-		(fields_autoplaced yes)
-		(effects
-			(font
-				(size 1.27 1.27)
-			)
-			(justify left)
-		)
-		(property "Intersheetrefs" "${INTERSHEET_REFS}"
-			(at 256.5618 66.04 0)
-			(hide yes)
-			(show_name no)
-			(do_not_autoplace no)
-			(effects
-				(font
-					(size 1.27 1.27)
-				)
-				(justify left)
-			)
-		)
-	)
 	(global_label "TR31"
 		(shape input)
@@
 		)
 	)
-	(global_label "TR12"
-		(shape input)
-		(at 120.65 67.31 0)
-		(fields_autoplaced yes)
-		(effects
-			(font
-				(size 1.27 1.27)
-			)
-			(justify left)
-		)
-		(property "Intersheetrefs" "${INTERSHEET_REFS}"
-			(at 128.2918 67.31 0)
-			(hide yes)
-			(show_name no)
-			(do_not_autoplace no)
-			(effects
-				(font
-					(size 1.27 1.27)
-				)
-				(justify left)
-			)
-		)
-	)
 	(global_label "ROWD"
 		(shape input)
@@
 		)
 	)
-	(global_label "TR22"
-		(shape input)
-		(at 120.65 72.39 0)
-		(fields_autoplaced yes)
-		(effects
-			(font
-				(size 1.27 1.27)
-			)
-			(justify left)
-		)
-		(property "Intersheetrefs" "${INTERSHEET_REFS}"
-			(at 128.2918 72.39 0)
-			(hide yes)
-			(show_name no)
-			(do_not_autoplace no)
-			(effects
-				(font
-					(size 1.27 1.27)
-				)
-				(justify left)
-			)
-		)
-	)
 	(global_label "TR11"
 		(shape input)
@@
 			)
 		)
-	)
-	(global_label "TR42"
-		(shape input)
-		(at 248.92 71.12 0)
-		(fields_autoplaced yes)
-		(effects
-			(font
-				(size 1.27 1.27)
-			)
-			(justify left)
-		)
-		(property "Intersheetrefs" "${INTERSHEET_REFS}"
-			(at 256.5618 71.12 0)
-			(hide yes)
-			(show_name no)
-			(do_not_autoplace no)
-			(effects
-				(font
-					(size 1.27 1.27)
-				)
-				(justify left)
-			)
-		)
