File: LED3 _BANK3.kicad_sch (KiCad schematic)
At the start: 76 parts, among them U7 STP16CPC26T

Commit message: update pcb
Connections:
- net C1_1: now also U7.20 (~{OUT15}); no longer U7.5 (~{OUT0})
- net C1_10: now also U7.11 (~{OUT6}); no longer U7.14 (~{OUT9})
- net C1_11: now also U7.10 (~{OUT5}); no longer U7.15 (~{OUT10})
- net C1_12: now also U7.9 (~{OUT4}); no longer U7.16 (~{OUT11})
- net C1_13: now also U7.8 (~{OUT3}); no longer U7.17 (~{OUT12})
- net C1_14: now also U7.7 (~{OUT2}); no longer U7.18 (~{OUT13})
- net C1_15: now also U7.6 (~{OUT1}); no longer U7.19 (~{OUT14})
- net C1_16: now also U7.5 (~{OUT0}); no longer U7.20 (~{OUT15})
- net C1_2: now also U7.19 (~{OUT14}); no longer U7.6 (~{OUT1})
- net C1_3: now also U7.18 (~{OUT13}); no longer U7.7 (~{OUT2})
- net C1_4: now also U7.17 (~{OUT12}); no longer U7.8 (~{OUT3})
- net C1_5: now also U7.16 (~{OUT11}); no longer U7.9 (~{OUT4})
- net C1_6: now also U7.15 (~{OUT10}); no longer U7.10 (~{OUT5})
- net C1_7: now also U7.14 (~{OUT9}); no longer U7.11 (~{OUT6})
- net C1_8: now also U7.13 (~{OUT8}); no longer U7.12 (~{OUT7})
- net C1_9: now also U7.12 (~{OUT7}); no longer U7.13 (~{OUT8})
Changed lines of the file:
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@@
 		)
 	)
-	(label "C1_13"
+	(label "C1_4"
 		(at 114.3 175.26 0)
 		(effects
@@
 		)
 	)
-	(label "C1_15"
+	(label "C1_2"
 		(at 114.3 180.34 0)
 		(effects
@@
 		)
 	)
-	(label "C1_3"
+	(label "C1_14"
 		(at 114.3 149.86 0)
 		(effects
@@
 		)
 	)
-	(label "C1_7"
+	(label "C1_10"
 		(at 114.3 160.02 0)
 		(effects
@@
 		)
 	)
-	(label "C1_6"
+	(label "C1_11"
 		(at 114.3 157.48 0)
 		(effects
@@
 		)
 	)
-	(label "C1_16"
+	(label "C1_1"
 		(at 114.3 182.88 0)
 		(effects
@@
 		)
 	)
-	(label "C1_11"
+	(label "C1_6"
 		(at 114.3 170.18 0)
 		(effects
@@
 		)
 	)
-	(label "C1_9"
+	(label "C1_8"
 		(at 114.3 165.1 0)
 		(effects
@@
 		)
 	)
-	(label "C1_4"
+	(label "C1_13"
 		(at 114.3 152.4 0)
 		(effects
@@
 		)
 	)
-	(label "C1_5"
+	(label "C1_12"
 		(at 114.3 154.94 0)
 		(effects
@@
 		)
 	)
-	(label "C1_8"
+	(label "C1_9"
 		(at 114.3 162.56 0)
 		(effects
@@
 		)
 	)
-	(label "C1_2"
+	(label "C1_15"
 		(at 114.3 147.32 0)
 		(effects
@@
 		)
 	)
-	(label "C1_14"
+	(label "C1_3"
 		(at 114.3 177.8 0)
 		(effects
@@
 		)
 	)
-	(label "C1_10"
+	(label "C1_7"
 		(at 114.3 167.64 0)
 		(effects
@@
 		)
 	)
-	(label "C1_1"
+	(label "C1_16"
 		(at 114.3 144.78 0)
 		(effects
@@
 		)
 	)
-	(label "C1_12"
+	(label "C1_5"
 		(at 114.3 172.72 0)
 		(effects
