File: LED4 _BANK4.kicad_sch (KiCad schematic)
At the start: 76 parts, among them U8 STP16CPC26T

Commit message: update pcb
Connections:
- net C1_1: now also U8.20 (~{OUT15}); no longer U8.5 (~{OUT0})
- net C1_10: now also U8.11 (~{OUT6}); no longer U8.14 (~{OUT9})
- net C1_11: now also U8.10 (~{OUT5}); no longer U8.15 (~{OUT10})
- net C1_12: now also U8.9 (~{OUT4}); no longer U8.16 (~{OUT11})
- net C1_13: now also U8.8 (~{OUT3}); no longer U8.17 (~{OUT12})
- net C1_14: now also U8.7 (~{OUT2}); no longer U8.18 (~{OUT13})
- net C1_15: now also U8.6 (~{OUT1}); no longer U8.19 (~{OUT14})
- net C1_16: now also U8.5 (~{OUT0}); no longer U8.20 (~{OUT15})
- net C1_2: now also U8.19 (~{OUT14}); no longer U8.6 (~{OUT1})
- net C1_3: now also U8.18 (~{OUT13}); no longer U8.7 (~{OUT2})
- net C1_4: now also U8.17 (~{OUT12}); no longer U8.8 (~{OUT3})
- net C1_5: now also U8.16 (~{OUT11}); no longer U8.9 (~{OUT4})
- net C1_6: now also U8.15 (~{OUT10}); no longer U8.10 (~{OUT5})
- net C1_7: now also U8.14 (~{OUT9}); no longer U8.11 (~{OUT6})
- net C1_8: now also U8.13 (~{OUT8}); no longer U8.12 (~{OUT7})
- net C1_9: now also U8.12 (~{OUT7}); no longer U8.13 (~{OUT8})
Changed lines of the file:
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@@
 		)
 	)
-	(label "C1_13"
+	(label "C1_4"
 		(at 113.03 175.26 0)
 		(effects
@@
 		)
 	)
-	(label "C1_2"
+	(label "C1_15"
 		(at 113.03 147.32 0)
 		(effects
@@
 		)
 	)
-	(label "C1_5"
+	(label "C1_12"
 		(at 113.03 154.94 0)
 		(effects
@@
 		)
 	)
-	(label "C1_7"
+	(label "C1_10"
 		(at 113.03 160.02 0)
 		(effects
@@
 		)
 	)
-	(label "C1_3"
+	(label "C1_14"
 		(at 113.03 149.86 0)
 		(effects
@@
 		)
 	)
-	(label "C1_15"
+	(label "C1_2"
 		(at 113.03 180.34 0)
 		(effects
@@
 		)
 	)
-	(label "C1_6"
+	(label "C1_11"
 		(at 113.03 157.48 0)
 		(effects
@@
 		)
 	)
-	(label "C1_10"
+	(label "C1_7"
 		(at 113.03 167.64 0)
 		(effects
@@
 		)
 	)
-	(label "C1_1"
+	(label "C1_16"
 		(at 113.03 144.78 0)
 		(effects
@@
 		)
 	)
-	(label "C1_16"
+	(label "C1_1"
 		(at 113.03 182.88 0)
 		(effects
@@
 		)
 	)
-	(label "C1_14"
+	(label "C1_3"
 		(at 113.03 177.8 0)
 		(effects
@@
 		)
 	)
-	(label "C1_4"
+	(label "C1_13"
 		(at 113.03 152.4 0)
 		(effects
@@
 		)
 	)
-	(label "C1_11"
+	(label "C1_6"
 		(at 113.03 170.18 0)
 		(effects
@@
 		)
 	)
-	(label "C1_8"
+	(label "C1_9"
 		(at 113.03 162.56 0)
 		(effects
@@
 		)
 	)
-	(label "C1_12"
+	(label "C1_5"
 		(at 113.03 172.72 0)
 		(effects
@@
 		)
 	)
-	(label "C1_9"
+	(label "C1_8"
 		(at 113.03 165.1 0)
 		(effects
