File: LEDS_BANK1.kicad_sch (KiCad schematic)
At the start: 76 parts, among them U1 STP16CPC26T

Commit message: update pcb
Connections:
- net C1_1: now also U1.20 (~{OUT15}); no longer U1.5 (~{OUT0})
- net C1_10: now also U1.11 (~{OUT6}); no longer U1.14 (~{OUT9})
- net C1_11: now also U1.10 (~{OUT5}); no longer U1.15 (~{OUT10})
- net C1_12: now also U1.9 (~{OUT4}); no longer U1.16 (~{OUT11})
- net C1_13: now also U1.8 (~{OUT3}); no longer U1.17 (~{OUT12})
- net C1_14: now also U1.7 (~{OUT2}); no longer U1.18 (~{OUT13})
- net C1_15: now also U1.6 (~{OUT1}); no longer U1.19 (~{OUT14})
- net C1_16: now also U1.5 (~{OUT0}); no longer U1.20 (~{OUT15})
- net C1_2: now also U1.19 (~{OUT14}); no longer U1.6 (~{OUT1})
- net C1_3: now also U1.18 (~{OUT13}); no longer U1.7 (~{OUT2})
- net C1_4: now also U1.17 (~{OUT12}); no longer U1.8 (~{OUT3})
- net C1_5: now also U1.16 (~{OUT11}); no longer U1.9 (~{OUT4})
- net C1_6: now also U1.15 (~{OUT10}); no longer U1.10 (~{OUT5})
- net C1_7: now also U1.14 (~{OUT9}); no longer U1.11 (~{OUT6})
- net C1_8: now also U1.13 (~{OUT8}); no longer U1.12 (~{OUT7})
- net C1_9: now also U1.12 (~{OUT7}); no longer U1.13 (~{OUT8})
Changed lines of the file:
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@@
 		)
 	)
-	(label "C1_2"
+	(label "C1_15"
 		(at 114.3 146.05 0)
 		(effects
@@
 		)
 	)
-	(label "C1_11"
+	(label "C1_6"
 		(at 114.3 168.91 0)
 		(effects
@@
 		)
 	)
-	(label "C1_9"
+	(label "C1_8"
 		(at 114.3 163.83 0)
 		(effects
@@
 		)
 	)
-	(label "C1_12"
+	(label "C1_5"
 		(at 114.3 171.45 0)
 		(effects
@@
 		)
 	)
-	(label "C1_5"
+	(label "C1_12"
 		(at 114.3 153.67 0)
 		(effects
@@
 		)
 	)
-	(label "C1_14"
+	(label "C1_3"
 		(at 114.3 176.53 0)
+		(effects
+			(font
+				(size 1.27 1.27)
+			)
+			(justify left bottom)
+		)
+	)
+	(label "C1_16"
+		(at 114.3 143.51 0)
+		(effects
+			(font
+				(size 1.27 1.27)
+			)
+			(justify left bottom)
+		)
+	)
+	(label "C1_16"
+		(at 114.3 143.51 0)
 		(effects
 			(font
@@
 		)
 	)
-	(label "C1_8"
+	(label "C1_9"
 		(at 114.3 161.29 0)
 		(effects
@@
 		)
 	)
-	(label "C1_4"
+	(label "C1_13"
 		(at 114.3 151.13 0)
 		(effects
@@
 		)
 	)
-	(label "C1_13"
+	(label "C1_4"
 		(at 114.3 173.99 0)
 		(effects
@@
 		)
 	)
-	(label "C1_10"
+	(label "C1_7"
 		(at 114.3 166.37 0)
 		(effects
@@
 		)
 	)
-	(label "C1_16"
+	(label "C1_1"
 		(at 114.3 181.61 0)
 		(effects
@@
 		)
 	)
-	(label "C1_7"
+	(label "C1_10"
 		(at 114.3 158.75 0)
 		(effects
@@
 		)
 	)
-	(label "C1_1"
-		(at 114.3 143.51 0)
-		(effects
-			(font
-				(size 1.27 1.27)
-			)
-			(justify left bottom)
-		)
-	)
 	(label "C1_4"
 		(at 193.04 93.98 0)
@@
 		)
 	)
-	(label "C1_6"
+	(label "C1_11"
 		(at 114.3 156.21 0)
 		(effects
@@
 		)
 	)
-	(label "C1_15"
+	(label "C1_2"
 		(at 114.3 179.07 0)
 		(effects
@@
 		)
 	)
-	(label "C1_3"
+	(label "C1_14"
 		(at 114.3 148.59 0)
 		(effects
