File: LEDS _BANK3.kicad_sch (KiCad schematic)
At the start: 76 parts, among them U3 STP16CPC26T

Commit message: update pcb
Connections:
- net C1_1: now also U3.20 (~{OUT15}); no longer U3.5 (~{OUT0})
- net C1_10: now also U3.11 (~{OUT6}); no longer U3.14 (~{OUT9})
- net C1_11: now also U3.10 (~{OUT5}); no longer U3.15 (~{OUT10})
- net C1_12: now also U3.9 (~{OUT4}); no longer U3.16 (~{OUT11})
- net C1_13: now also U3.8 (~{OUT3}); no longer U3.17 (~{OUT12})
- net C1_14: now also U3.7 (~{OUT2}); no longer U3.18 (~{OUT13})
- net C1_15: now also U3.6 (~{OUT1}); no longer U3.19 (~{OUT14})
- net C1_16: now also U3.5 (~{OUT0}); no longer U3.20 (~{OUT15})
- net C1_2: now also U3.19 (~{OUT14}); no longer U3.6 (~{OUT1})
- net C1_3: now also U3.18 (~{OUT13}); no longer U3.7 (~{OUT2})
- net C1_4: now also U3.17 (~{OUT12}); no longer U3.8 (~{OUT3})
- net C1_5: now also U3.16 (~{OUT11}); no longer U3.9 (~{OUT4})
- net C1_6: now also U3.15 (~{OUT10}); no longer U3.10 (~{OUT5})
- net C1_7: now also U3.14 (~{OUT9}); no longer U3.11 (~{OUT6})
- net C1_8: now also U3.13 (~{OUT8}); no longer U3.12 (~{OUT7})
- net C1_9: now also U3.12 (~{OUT7}); no longer U3.13 (~{OUT8})
Changed lines of the file:
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@@
 		)
 	)
-	(label "C1_8"
+	(label "C1_9"
 		(at 114.3 162.56 0)
 		(effects
@@
 		)
 	)
-	(label "C1_15"
+	(label "C1_2"
 		(at 114.3 180.34 0)
 		(effects
@@
 		)
 	)
-	(label "C1_5"
+	(label "C1_12"
 		(at 114.3 154.94 0)
 		(effects
@@
 		)
 	)
-	(label "C1_1"
+	(label "C1_16"
 		(at 114.3 144.78 0)
 		(effects
@@
 		)
 	)
-	(label "C1_11"
+	(label "C1_6"
 		(at 114.3 170.18 0)
 		(effects
@@
 		)
 	)
-	(label "C1_9"
+	(label "C1_8"
 		(at 114.3 165.1 0)
 		(effects
@@
 		)
 	)
-	(label "C1_4"
+	(label "C1_13"
 		(at 114.3 152.4 0)
 		(effects
@@
 		)
 	)
-	(label "C1_14"
+	(label "C1_3"
 		(at 114.3 177.8 0)
 		(effects
@@
 		)
 	)
-	(label "C1_6"
+	(label "C1_11"
 		(at 114.3 157.48 0)
 		(effects
@@
 		)
 	)
-	(label "C1_12"
+	(label "C1_5"
 		(at 114.3 172.72 0)
 		(effects
@@
 		)
 	)
-	(label "C1_2"
+	(label "C1_15"
 		(at 114.3 147.32 0)
 		(effects
@@
 		)
 	)
-	(label "C1_16"
+	(label "C1_1"
 		(at 114.3 182.88 0)
 		(effects
@@
 		)
 	)
-	(label "C1_7"
+	(label "C1_10"
 		(at 114.3 160.02 0)
 		(effects
@@
 		)
 	)
-	(label "C1_10"
+	(label "C1_7"
 		(at 114.3 167.64 0)
 		(effects
@@
 		)
 	)
-	(label "C1_13"
+	(label "C1_4"
 		(at 114.3 175.26 0)
 		(effects
@@
 		)
 	)
-	(label "C1_3"
+	(label "C1_14"
 		(at 114.3 149.86 0)
 		(effects

Commit message: Initial KiCad project
Parts:
- renumbered DC28 to DC25, DC30 to DC26, DC31 to DC27, DC27 to DC28, DC25 to DC30, DC32 to DC31, DC33 to DC32, DC26 to DC33
Changed lines of the file:
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@@
 		(dnp no)
 		(fields_autoplaced yes)
-		(property "Reference" "DC25"
+		(property "Reference" "DC30"
 			(at 26.67 82.6769 0)
 			(show_name no)
@@
 			(project "P10_LED_2"
 				(path "/5bf83443-a365-405c-87ec-0622411c2f24/cb31e7ee-8e0a-4a9d-a2fd-a754182503d6"
-					(reference "DC25")
+					(reference "DC30")
 					(unit 1)
 				)
@@
 		(dnp no)
 		(fields_autoplaced yes)
-		(property "Reference" "DC28"
+		(property "Reference" "DC25"
 			(at 29.21 28.0669 0)
 			(show_name no)
@@
 			(project "P10_LED_2"
 				(path "/5bf83443-a365-405c-87ec-0622411c2f24/cb31e7ee-8e0a-4a9d-a2fd-a754182503d6"
-					(reference "DC28")
+					(reference "DC25")
 					(unit 1)
 				)
@@
 		(dnp no)
 		(fields_autoplaced yes)
-		(property "Reference" "DC26"
+		(property "Reference" "DC33"
 			(at 26.67 113.1569 0)
 			(show_name no)
@@
 			(project "P10_LED_2"
 				(path "/5bf83443-a365-405c-87ec-0622411c2f24/cb31e7ee-8e0a-4a9d-a2fd-a754182503d6"
-					(reference "DC26")
+					(reference "DC33")
 					(unit 1)
 				)
@@
 		(dnp no)
 		(fields_autoplaced yes)
-		(property "Reference" "DC27"
+		(property "Reference" "DC28"
 			(at 27.94 56.0069 0)
 			(show_name no)
@@
 			(project "P10_LED_2"
 				(path "/5bf83443-a365-405c-87ec-0622411c2f24/cb31e7ee-8e0a-4a9d-a2fd-a754182503d6"
-					(reference "DC27")
+					(reference "DC28")
 					(unit 1)
 				)
@@
 		(dnp no)
 		(fields_autoplaced yes)
-		(property "Reference" "DC33"
+		(property "Reference" "DC32"
 			(at 250.19 111.8869 0)
 			(show_name no)
@@
 			(project "P10_LED_2"
 				(path "/5bf83443-a365-405c-87ec-0622411c2f24/cb31e7ee-8e0a-4a9d-a2fd-a754182503d6"
-					(reference "DC33")
+					(reference "DC32")
 					(unit 1)
 				)
@@
 		(dnp no)
 		(fields_autoplaced yes)
-		(property "Reference" "DC30"
+		(property "Reference" "DC26"
 			(at 250.19 28.0669 0)
 			(show_name no)
@@
 			(project "P10_LED_2"
 				(path "/5bf83443-a365-405c-87ec-0622411c2f24/cb31e7ee-8e0a-4a9d-a2fd-a754182503d6"
-					(reference "DC30")
+					(reference "DC26")
 					(unit 1)
 				)
@@
 		(dnp no)
 		(fields_autoplaced yes)
-		(property "Reference" "DC31"
+		(property "Reference" "DC27"
 			(at 250.19 54.7369 0)
 			(show_name no)
@@
 			(project "P10_LED_2"
 				(path "/5bf83443-a365-405c-87ec-0622411c2f24/cb31e7ee-8e0a-4a9d-a2fd-a754182503d6"
-					(reference "DC31")
+					(reference "DC27")
 					(unit 1)
 				)
@@
 		(dnp no)
 		(fields_autoplaced yes)
-		(property "Reference" "DC32"
+		(property "Reference" "DC31"
 			(at 250.19 82.6769 0)
 			(show_name no)
@@
 			(project "P10_LED_2"
 				(path "/5bf83443-a365-405c-87ec-0622411c2f24/cb31e7ee-8e0a-4a9d-a2fd-a754182503d6"
-					(reference "DC32")
+					(reference "DC31")
 					(unit 1)
 				)
