File: P10_LED_2.kicad_pcb (KiCad board)
At the start: 2 copper layers, 297.6 x 218.3 mm, 710 parts, among them J1 2 Pin 5.5mm Male Molex OUTPUT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, J2 2 Pin 5.5mm Male Molex INPUT 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, J3 2 Pin 5.5mm Male Molex MAINS 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, J4 5 PIN 2.54MM PITCH BURGSTRIP, J5 5-PIN 2.54MM PITCH MALE STRAI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, J6 5-PIN 2.54MM PITCH MALE STRAI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, J7 Conn_02x07_Odd_Even, J8 Conn_02x07_Odd_Even, SW1 SW_DIP_x04, U1 STP16CPC26T, U10 STM32401VBT6 100 PIN LQFP, U11 MAX3483, U12 MX25L6406EM21, U2 STP16CPC26T, U3 STP16CPC26T, U4 STP16CPC26T, U5 STP16CPC26T, U6 STP16CPC26T, U7 STP16CPC26T, U8 STP16CPC26T, U9 MP24943DN-LF-Z SOIC8E

Commit message: update pcb
Parts:
- added U14: ~, Package_SO:SOIC-8_3.9x4.9mm_P1.27mm, B.Cu at (916.8, 321.0)
- C28, C29, C30, C31, C32, C33, C34, C35, DC10, DC11, DC12, DC13, DC14, DC15, DC16, DC17, DC18, DC19, DC20, DC21, DC25, DC26, DC27, DC28, DC30, DC31, DC32, DC33, DC34, DC35, DC36, DC37, DC38, DC39, DC4, DC40, DC41, DC44, DC45, DC46, DC47, DC48, DC49, DC5, DC50, DC51, DC54, DC55, DC56, DC57, DC58, DC59, DC6, DC60, DC61, DC64, DC65, DC66, DC67, DC68, DC69, DC7, DC70, DC71, DC74, DC75, DC76, DC77, DC78, DC79, DC8, DC80, DC81, DC9, R25, R26, R27, R28, R29, U1, U13, U2, U3, U4, U5, U6, U7, U8: moved to B.Cu
- moved U10 431.1 mm to (890.2, 272.7)
- moved R27 333.5 mm to (947.1, 318.7), turned to -90 degrees
- moved R28 333.5 mm to (944.7, 318.4), turned to -90 degrees
- moved R25 312.8 mm to (928.7, 318.2), turned to 90 degrees
- moved R26 311.3 mm to (925.0, 318.2), turned to 90 degrees
- moved DC7 304.3 mm to (969.7, 319.9), turned to -90 degrees
- moved DC27 303.3 mm to (968.0, 430.8), turned to 180 degrees
- moved DC4 303.0 mm to (968.6, 308.2), turned to 180 degrees
- moved DC28 302.9 mm to (967.5, 416.5), turned to 180 degrees
- moved DC11 302.7 mm to (968.1, 351.1), turned to 180 degrees
- moved DC17 302.6 mm to (968.2, 376.1), turned to 180 degrees
- moved DC8 302.6 mm to (968.4, 334.0), turned to 180 degrees
- moved DC18 302.5 mm to (968.0, 389.8), turned to 180 degrees
- moved DC14 302.4 mm to (968.2, 362.6), turned to 180 degrees
- moved DC21 302.3 mm to (968.1, 402.2), turned to 180 degrees
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Connections:
- U1 pad 10: /LEDS_BANK1/C1_6 -> /LEDS_BANK1/C1_11
- U1 pad 11: /LEDS_BANK1/C1_7 -> /LEDS_BANK1/C1_10
- U1 pad 12: /LEDS_BANK1/C1_8 -> /LEDS_BANK1/C1_9
- U1 pad 13: /LEDS_BANK1/C1_9 -> /LEDS_BANK1/C1_8
- U1 pad 14: /LEDS_BANK1/C1_10 -> /LEDS_BANK1/C1_7
- U1 pad 15: /LEDS_BANK1/C1_11 -> /LEDS_BANK1/C1_6
- U1 pad 16: /LEDS_BANK1/C1_12 -> /LEDS_BANK1/C1_5
- U1 pad 17: /LEDS_BANK1/C1_13 -> /LEDS_BANK1/C1_4
- U1 pad 18: /LEDS_BANK1/C1_14 -> /LEDS_BANK1/C1_3
- U1 pad 19: /LEDS_BANK1/C1_15 -> /LEDS_BANK1/C1_2
- U1 pad 20: /LEDS_BANK1/C1_16 -> /LEDS_BANK1/C1_1
- U1 pad 5: /LEDS_BANK1/C1_1 -> /LEDS_BANK1/C1_16
- U1 pad 6: /LEDS_BANK1/C1_2 -> /LEDS_BANK1/C1_15
- U1 pad 7: /LEDS_BANK1/C1_3 -> /LEDS_BANK1/C1_14
- U1 pad 8: /LEDS_BANK1/C1_4 -> /LEDS_BANK1/C1_13
- U1 pad 9: /LEDS_BANK1/C1_5 -> /LEDS_BANK1/C1_12
- U2 pad 10: /LEDS_BANK2/C1_6 -> /LEDS_BANK2/C1_11
- U2 pad 11: /LEDS_BANK2/C1_7 -> /LEDS_BANK2/C1_10
- U2 pad 12: /LEDS_BANK2/C1_8 -> /LEDS_BANK2/C1_9
- U2 pad 13: /LEDS_BANK2/C1_9 -> /LEDS_BANK2/C1_8
- U2 pad 14: /LEDS_BANK2/C1_10 -> /LEDS_BANK2/C1_7
- U2 pad 15: /LEDS_BANK2/C1_11 -> /LEDS_BANK2/C1_6
- U2 pad 16: /LEDS_BANK2/C1_12 -> /LEDS_BANK2/C1_5
- U2 pad 17: /LEDS_BANK2/C1_13 -> /LEDS_BANK2/C1_4
- U2 pad 18: /LEDS_BANK2/C1_14 -> /LEDS_BANK2/C1_3
- U2 pad 19: /LEDS_BANK2/C1_15 -> /LEDS_BANK2/C1_2
- U2 pad 20: /LEDS_BANK2/C1_16 -> /LEDS_BANK2/C1_1
- U2 pad 5: /LEDS_BANK2/C1_1 -> /LEDS_BANK2/C1_16
- U2 pad 6: /LEDS_BANK2/C1_2 -> /LEDS_BANK2/C1_15
- U2 pad 7: /LEDS_BANK2/C1_3 -> /LEDS_BANK2/C1_14
- U2 pad 8: /LEDS_BANK2/C1_4 -> /LEDS_BANK2/C1_13
- U2 pad 9: /LEDS_BANK2/C1_5 -> /LEDS_BANK2/C1_12
- U3 pad 10: /LEDS _BANK3/C1_6 -> /LEDS _BANK3/C1_11
- U3 pad 11: /LEDS _BANK3/C1_7 -> /LEDS _BANK3/C1_10
- U3 pad 12: /LEDS _BANK3/C1_8 -> /LEDS _BANK3/C1_9
- U3 pad 13: /LEDS _BANK3/C1_9 -> /LEDS _BANK3/C1_8
- U3 pad 14: /LEDS _BANK3/C1_10 -> /LEDS _BANK3/C1_7
- U3 pad 15: /LEDS _BANK3/C1_11 -> /LEDS _BANK3/C1_6
- U3 pad 16: /LEDS _BANK3/C1_12 -> /LEDS _BANK3/C1_5
- U3 pad 17: /LEDS _BANK3/C1_13 -> /LEDS _BANK3/C1_4
- U3 pad 18: /LEDS _BANK3/C1_14 -> /LEDS _BANK3/C1_3
- U3 pad 19: /LEDS _BANK3/C1_15 -> /LEDS _BANK3/C1_2
- U3 pad 20: /LEDS _BANK3/C1_16 -> /LEDS _BANK3/C1_1
- U3 pad 5: /LEDS _BANK3/C1_1 -> /LEDS _BANK3/C1_16
- U3 pad 6: /LEDS _BANK3/C1_2 -> /LEDS _BANK3/C1_15
- U3 pad 7: /LEDS _BANK3/C1_3 -> /LEDS _BANK3/C1_14
- U3 pad 8: /LEDS _BANK3/C1_4 -> /LEDS _BANK3/C1_13
- U3 pad 9: /LEDS _BANK3/C1_5 -> /LEDS _BANK3/C1_12
- U4 pad 10: /LEDS _BANK4 (page 11)/C1_6 -> /LEDS _BANK4 (page 11)/C1_11
- U4 pad 11: /LEDS _BANK4 (page 11)/C1_7 -> /LEDS _BANK4 (page 11)/C1_10
- U4 pad 12: /LEDS _BANK4 (page 11)/C1_8 -> /LEDS _BANK4 (page 11)/C1_9
- U4 pad 13: /LEDS _BANK4 (page 11)/C1_9 -> /LEDS _BANK4 (page 11)/C1_8
- U4 pad 14: /LEDS _BANK4 (page 11)/C1_10 -> /LEDS _BANK4 (page 11)/C1_7
- U4 pad 15: /LEDS _BANK4 (page 11)/C1_11 -> /LEDS _BANK4 (page 11)/C1_6
- U4 pad 16: /LEDS _BANK4 (page 11)/C1_12 -> /LEDS _BANK4 (page 11)/C1_5
- U4 pad 17: /LEDS _BANK4 (page 11)/C1_13 -> /LEDS _BANK4 (page 11)/C1_4
- U4 pad 18: /LEDS _BANK4 (page 11)/C1_14 -> /LEDS _BANK4 (page 11)/C1_3
- U4 pad 19: /LEDS _BANK4 (page 11)/C1_15 -> /LEDS _BANK4 (page 11)/C1_2
- U4 pad 20: /LEDS _BANK4 (page 11)/C1_16 -> /LEDS _BANK4 (page 11)/C1_1
- U4 pad 5: /LEDS _BANK4 (page 11)/C1_1 -> /LEDS _BANK4 (page 11)/C1_16
- U4 pad 6: /LEDS _BANK4 (page 11)/C1_2 -> /LEDS _BANK4 (page 11)/C1_15
- U4 pad 7: /LEDS _BANK4 (page 11)/C1_3 -> /LEDS _BANK4 (page 11)/C1_14
- U4 pad 8: /LEDS _BANK4 (page 11)/C1_4 -> /LEDS _BANK4 (page 11)/C1_13
- U4 pad 9: /LEDS _BANK4 (page 11)/C1_5 -> /LEDS _BANK4 (page 11)/C1_12
- U5 pad 10: /LED1 _BANK1/C1_6 -> /LED1 _BANK1/C1_11
- U5 pad 11: /LED1 _BANK1/C1_7 -> /LED1 _BANK1/C1_10
- U5 pad 12: /LED1 _BANK1/C1_8 -> /LED1 _BANK1/C1_9
- U5 pad 13: /LED1 _BANK1/C1_9 -> /LED1 _BANK1/C1_8
- U5 pad 14: /LED1 _BANK1/C1_10 -> /LED1 _BANK1/C1_7
- U5 pad 15: /LED1 _BANK1/C1_11 -> /LED1 _BANK1/C1_6
- U5 pad 16: /LED1 _BANK1/C1_12 -> /LED1 _BANK1/C1_5
- U5 pad 17: /LED1 _BANK1/C1_13 -> /LED1 _BANK1/C1_4
- U5 pad 18: /LED1 _BANK1/C1_14 -> /LED1 _BANK1/C1_3
- U5 pad 19: /LED1 _BANK1/C1_15 -> /LED1 _BANK1/C1_2
- U5 pad 20: /LED1 _BANK1/C1_16 -> /LED1 _BANK1/C1_1
- U5 pad 5: /LED1 _BANK1/C1_1 -> /LED1 _BANK1/C1_16
- U5 pad 6: /LED1 _BANK1/C1_2 -> /LED1 _BANK1/C1_15
- U5 pad 7: /LED1 _BANK1/C1_3 -> /LED1 _BANK1/C1_14
- U5 pad 8: /LED1 _BANK1/C1_4 -> /LED1 _BANK1/C1_13
- U5 pad 9: /LED1 _BANK1/C1_5 -> /LED1 _BANK1/C1_12
- U6 pad 10: /LED2_BANK2/C1_6 -> /LED2_BANK2/C1_11
- U6 pad 11: /LED2_BANK2/C1_7 -> /LED2_BANK2/C1_10
- U6 pad 12: /LED2_BANK2/C1_8 -> /LED2_BANK2/C1_9
- U6 pad 13: /LED2_BANK2/C1_9 -> /LED2_BANK2/C1_8
- U6 pad 14: /LED2_BANK2/C1_10 -> /LED2_BANK2/C1_7
- U6 pad 15: /LED2_BANK2/C1_11 -> /LED2_BANK2/C1_6
- U6 pad 16: /LED2_BANK2/C1_12 -> /LED2_BANK2/C1_5
- U6 pad 17: /LED2_BANK2/C1_13 -> /LED2_BANK2/C1_4
- U6 pad 18: /LED2_BANK2/C1_14 -> /LED2_BANK2/C1_3
- U6 pad 19: /LED2_BANK2/C1_15 -> /LED2_BANK2/C1_2
- U6 pad 20: /LED2_BANK2/C1_16 -> /LED2_BANK2/C1_1
- U6 pad 5: /LED2_BANK2/C1_1 -> /LED2_BANK2/C1_16
- U6 pad 6: /LED2_BANK2/C1_2 -> /LED2_BANK2/C1_15
- U6 pad 7: /LED2_BANK2/C1_3 -> /LED2_BANK2/C1_14
- U6 pad 8: /LED2_BANK2/C1_4 -> /LED2_BANK2/C1_13
- U6 pad 9: /LED2_BANK2/C1_5 -> /LED2_BANK2/C1_12
- U7 pad 10: /LED3 _BANK3/C1_6 -> /LED3 _BANK3/C1_11
- U7 pad 11: /LED3 _BANK3/C1_7 -> /LED3 _BANK3/C1_10
- U7 pad 12: /LED3 _BANK3/C1_8 -> /LED3 _BANK3/C1_9
- U7 pad 13: /LED3 _BANK3/C1_9 -> /LED3 _BANK3/C1_8
- U7 pad 14: /LED3 _BANK3/C1_10 -> /LED3 _BANK3/C1_7
- U7 pad 15: /LED3 _BANK3/C1_11 -> /LED3 _BANK3/C1_6
- U7 pad 16: /LED3 _BANK3/C1_12 -> /LED3 _BANK3/C1_5
- U7 pad 17: /LED3 _BANK3/C1_13 -> /LED3 _BANK3/C1_4
- U7 pad 18: /LED3 _BANK3/C1_14 -> /LED3 _BANK3/C1_3
- U7 pad 19: /LED3 _BANK3/C1_15 -> /LED3 _BANK3/C1_2
- U7 pad 20: /LED3 _BANK3/C1_16 -> /LED3 _BANK3/C1_1
- U7 pad 5: /LED3 _BANK3/C1_1 -> /LED3 _BANK3/C1_16
- U7 pad 6: /LED3 _BANK3/C1_2 -> /LED3 _BANK3/C1_15
- U7 pad 7: /LED3 _BANK3/C1_3 -> /LED3 _BANK3/C1_14
- U7 pad 8: /LED3 _BANK3/C1_4 -> /LED3 _BANK3/C1_13
- U7 pad 9: /LED3 _BANK3/C1_5 -> /LED3 _BANK3/C1_12
- U8 pad 10: /LED4 _BANK4/C1_6 -> /LED4 _BANK4/C1_11
- U8 pad 11: /LED4 _BANK4/C1_7 -> /LED4 _BANK4/C1_10
- U8 pad 12: /LED4 _BANK4/C1_8 -> /LED4 _BANK4/C1_9
- U8 pad 13: /LED4 _BANK4/C1_9 -> /LED4 _BANK4/C1_8
- U8 pad 14: /LED4 _BANK4/C1_10 -> /LED4 _BANK4/C1_7
- U8 pad 15: /LED4 _BANK4/C1_11 -> /LED4 _BANK4/C1_6
- U8 pad 16: /LED4 _BANK4/C1_12 -> /LED4 _BANK4/C1_5
- U8 pad 17: /LED4 _BANK4/C1_13 -> /LED4 _BANK4/C1_4
- U8 pad 18: /LED4 _BANK4/C1_14 -> /LED4 _BANK4/C1_3
- U8 pad 19: /LED4 _BANK4/C1_15 -> /LED4 _BANK4/C1_2
- U8 pad 20: /LED4 _BANK4/C1_16 -> /LED4 _BANK4/C1_1
- U8 pad 5: /LED4 _BANK4/C1_1 -> /LED4 _BANK4/C1_16
- U8 pad 6: /LED4 _BANK4/C1_2 -> /LED4 _BANK4/C1_15
- U8 pad 7: /LED4 _BANK4/C1_3 -> /LED4 _BANK4/C1_14
- U8 pad 8: /LED4 _BANK4/C1_4 -> /LED4 _BANK4/C1_13
- U8 pad 9: /LED4 _BANK4/C1_5 -> /LED4 _BANK4/C1_12
Routing:
- net TR21: track 0.00 -> 2121.2 mm, vias 0 -> 127
- net TR31: track 0.00 -> 2097.7 mm, vias 0 -> 124
- net TR41: track 0.00 -> 1963.7 mm, vias 0 -> 94
- net TR11: track 628.0 -> 1336.0 mm, vias 0 -> 1
- net GND: track 0.00 -> 143.7 mm, vias 0 -> 2
- net (no net): track 79.1 -> 2.65 mm, vias 1 -> 0
- net /LEDS_BANK1/C1_1: track 43.6 -> 119.9 mm, vias 0 -> 1
- net ROWB: track 0.00 -> 69.1 mm
- net ROWD: track 0.00 -> 58.4 mm
- net ROWC: track 0.00 -> 50.2 mm
- net VCC: track 0.00 -> 39.0 mm, vias 0 -> 2
- net ROWA: track 0.00 -> 28.9 mm
- net /LEDS _BANK3/C1_4: track 89.3 -> 64.4 mm
- net VCC_3V3_1: track 0.00 -> 18.7 mm
- net VCC_3V3_2: track 0.00 -> 18.7 mm
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
Commit message: Initial KiCad project
Parts:
- C1, C10, C11, C12, C13, C14, C15, C16, C17, C18, C19, C2, C20, C21, C22, C23, C24, C25, C26, C27, C3, C4, C5, C6, C7, C8, C9, D513, D514, D515, D516, D517, DC1, DC2, DC22, DC23, DC24, DC29, DC3, DC42, DC43, DC52, DC53, DC62, DC63, DC72, DC73, DC82, DC83, F1, F2, F3, F4, J1, J2, J3, J4, J5, J6, J7, J8, L1, L2, L2A1, L3, L4, L5, L6, L7, LDR1, NTC1, R1, R10, R11, R12, R13, R14, R15, R16, R17, R18, R19, R2, R20, R21, R22, R23, R24, R3, R30, R31, R32, R33, R34, R35, R36, R4, R5, R6, R7, R8, R9, RV1, RV2, RV3, SW1, U10, U11, U12, U9: moved to B.Cu
- DC25: value 1.8nF -> 1.8 nF
- DC26, DC27: value 1.8nF -> 0.01 uF
- DC28: value 1.8 nF -> 1.8nF
- DC30, DC33: value 0.01 uF -> 1.8nF
- moved NTC1 716.6 mm to (545.5, 25.3), turned to 180 degrees
- moved J8 682.4 mm to (515.2, 17.0), turned to 180 degrees
- moved LDR1 675.6 mm to (566.3, 24.8), turned to 180 degrees
- moved C27 594.5 mm to (604.7, 16.9), turned to 180 degrees
- moved C26 592.4 mm to (604.7, 13.6), turned to 180 degrees
- moved C25 571.1 mm to (607.8, 33.1), turned to 180 degrees
- moved J4 569.3 mm to (590.1, 19.7), turned to 180 degrees
- moved C24 568.9 mm to (608.0, 29.7), turned to 180 degrees
- moved C23 566.7 mm to (608.2, 26.4), turned to 180 degrees
- moved C22 564.0 mm to (608.2, 23.0), turned to 180 degrees
- moved L2A1 563.3 mm to (576.5, 265.5), turned to 180 degrees
- moved SW1 560.1 mm to (671.8, 23.4), turned to -90 degrees
- moved C16 556.7 mm to (577.4, 24.6), turned to 180 degrees
- moved D517 547.6 mm to (562.5, 275.7), turned to -90 degrees
- moved C21 533.2 mm to (643.5, 25.2), turned to -90 degrees
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Connections:
- DC25 pad 1: TR31 -> TR11
- DC26 pad 1: TR41 -> TR11
- DC28 pad 1: TR11 -> TR21
- DC30 pad 1: TR11 -> TR31
- DC31 pad 1: TR21 -> TR31
- DC32 pad 1: TR31 -> TR41
Routing:
- net TR21: track 2121.2 -> 0.00 mm, vias 127 -> 0
- net TR31: track 2097.7 -> 0.00 mm, vias 124 -> 0
- net TR41: track 1963.7 -> 0.00 mm, vias 94 -> 0
- net GND: track 143.7 -> 0.00 mm, vias 2 -> 0
- net /LEDS_BANK2/C1_1: track 120.1 -> 0.00 mm, vias 1 -> 0
- net /LEDS _BANK3/C1_1: track 121.6 -> 41.1 mm, vias 1 -> 0
- net TR11: track 1336.0 -> 1255.9 mm, vias 1 -> 0
- net /LEDS _BANK4 (page 11)/C1_1: track 120.3 -> 41.1 mm, vias 1 -> 0
- net /LEDS _BANK3/C1_16: track 120.2 -> 41.1 mm, vias 1 -> 0
- net /LEDS_BANK1/C1_1: track 119.9 -> 41.1 mm, vias 1 -> 0
- net /LEDS _BANK4 (page 11)/C1_16: track 119.6 -> 41.1 mm, vias 1 -> 0
- net /LED1 _BANK1/C1_1: track 119.3 -> 41.1 mm, vias 1 -> 0
- net /LEDS_BANK1/C1_16: track 119.2 -> 41.1 mm, vias 1 -> 0
- net /LED2_BANK2/C1_1: track 118.8 -> 41.1 mm, vias 1 -> 0
- net /LED4 _BANK4/C1_16: track 118.3 -> 41.1 mm, vias 1 -> 0
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Other:
- board outline removed

Commit message: updated pcb
Parts:
- moved DC2 32.1 mm to (773.1, 11.0)
- moved DC3 31.9 mm to (773.1, 14.9)
- moved R34 27.8 mm to (588.0, 146.9), turned to 0 degrees
- moved R32 27.6 mm to (736.5, 256.8), turned to 0 degrees
- moved R35 27.2 mm to (587.3, 201.7), turned to 0 degrees
- moved R33 26.8 mm to (586.9, 91.8), turned to 0 degrees
- moved R31 26.6 mm to (735.2, 201.8), turned to 0 degrees
- moved R36 26.4 mm to (586.4, 256.7), turned to 0 degrees
- moved R30 26.1 mm to (734.9, 146.3), turned to 0 degrees
- moved R29 24.4 mm to (734.5, 91.7), turned to 0 degrees
- moved DC42 22.4 mm to (731.6, 256.8), turned to 0 degrees
- moved DC62 22.3 mm to (583.0, 146.9), turned to 0 degrees
- moved DC29 22.1 mm to (730.8, 201.9), turned to 0 degrees
- moved DC72 21.8 mm to (582.7, 201.7), turned to 0 degrees
- moved DC52 21.5 mm to (582.1, 91.8), turned to 0 degrees
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Routing:
- net TR21: track 0.00 -> 1766.9 mm, vias 0 -> 142
- net TR31: track 0.00 -> 1763.1 mm, vias 0 -> 142
- net GND: track 0.00 -> 1499.5 mm, vias 0 -> 6
- net TR41: track 0.00 -> 1404.1 mm, vias 0 -> 8
- net GNDREF: track 0.00 -> 377.3 mm, vias 0 -> 2
- net VCC_3V3_1: track 0.00 -> 346.5 mm, vias 0 -> 4
- net VCC_24V_OUT: track 0.00 -> 321.1 mm
- net SPI_MOSI: track 0.00 -> 176.3 mm, vias 0 -> 4
- net ROWC: track 0.00 -> 171.4 mm
- net ROWA: track 0.00 -> 171.3 mm
- net DATA_1_IN: track 0.00 -> 170.6 mm
- net DATA_3_IN: track 0.00 -> 169.6 mm
- net ROWB: track 0.00 -> 168.8 mm
- net ROWD: track 0.00 -> 168.7 mm
- net LATCH: track 0.00 -> 167.6 mm
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