File: P10_LED_2.kicad_pcb (KiCad board)
At the start: 2 copper layers, 711 parts, among them J1 2 Pin 5.5mm Male Molex OUTPUT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, J2 2 Pin 5.5mm Male Molex INPUT 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, J3 2 Pin 5.5mm Male Molex MAINS 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, J4 5 PIN 2.54MM PITCH BURGSTRIP, J5 5-PIN 2.54MM PITCH MALE STRAI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, J6 5-PIN 2.54MM PITCH MALE STRAI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, J7 Conn_02x07_Odd_Even, J8 Conn_02x07_Odd_Even, SW1 SW_DIP_x04, U1 STP16CPC26T, U10 STM32401VBT6 100 PIN LQFP, U11 MAX3483, U12 MX25L6406EM21, U2 STP16CPC26T, U3 STP16CPC26T, U4 STP16CPC26T, U5 STP16CPC26T, U6 STP16CPC26T, U7 STP16CPC26T, U8 STP16CPC26T, U9 MP24943DN-LF-Z SOIC8E

Commit message: updated pcb
Parts:
- moved R25 4.41 mm to (619.6, 181.6)
- moved R26 3.58 mm to (619.6, 185.5)
- moved C17 2.43 mm to (632.4, 13.5)
- moved R12 2.08 mm to (627.0, 13.4)
- moved R13 2.08 mm to (627.0, 11.0)
Routing:
- net ROWC: track 171.4 -> 321.1 mm, vias 0 -> 1
- net ROWA: track 171.3 -> 318.2 mm, vias 0 -> 1
- net ROWB: track 168.8 -> 309.7 mm, vias 0 -> 1
- net ROWD: track 168.7 -> 307.6 mm, vias 0 -> 1
- net SPI_SCLK: track 0.00 -> 138.8 mm, vias 0 -> 6
- net SPI_NSS: track 0.00 -> 131.6 mm, vias 0 -> 6
- net TR21: track 1766.9 -> 1862.4 mm, vias 142 -> 154
- net VCC_3V3_1: track 346.5 -> 441.1 mm, vias 4 -> 6
- net TR11: track 1320.2 -> 1408.8 mm, vias 7 -> 17
- net AIN_1: track 21.9 -> 110.3 mm, vias 0 -> 1
- net AIN_2: track 15.6 -> 87.6 mm, vias 0 -> 3
- net TR31: track 1763.1 -> 1830.3 mm, vias 142 -> 151
- net TR41: track 1404.1 -> 1467.6 mm, vias 8 -> 18
- net SW_8: track 5.67 -> 68.4 mm, vias 0 -> 2
- net SW_4: track 4.82 -> 64.9 mm, vias 0 -> 2
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
Commit message: update
Routing:
- net OE: track 164.7 -> 801.9 mm, vias 0 -> 17
- net LATCH: track 167.6 -> 775.2 mm, vias 0 -> 19
- net SCLK: track 165.7 -> 764.0 mm, vias 0 -> 17
- net DATA_1: track 0.00 -> 156.4 mm, vias 0 -> 2
- net DATA_1_IN: track 170.6 -> 316.4 mm, vias 0 -> 3
- net GND: track 1511.2 -> 1497.8 mm, vias 6 -> 18
- net /LEDS _BANK3/C1_9: track 41.1 -> 50.4 mm, vias 0 -> 1
- net /LED4 _BANK4/C1_11: track 69.9 -> 67.4 mm
- net /LED3 _BANK3/C1_11: track 70.6 -> 68.4 mm
- net /LED4 _BANK4/C1_12: track 79.7 -> 77.6 mm
- net /LED4 _BANK4/C1_13: track 88.0 -> 86.0 mm
- net /LED4 _BANK4/C1_14: track 98.2 -> 96.6 mm
- net /LED3 _BANK3/C1_12: track 78.8 -> 77.5 mm
- net /LEDS _BANK4 (page 11)/C1_11: track 69.7 -> 68.7 mm
- net /LED1 _BANK1/C1_9: track 48.0 -> 47.3 mm
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
Commit message: updated
Routing:
- net VCC: track 93.2 -> 607.0 mm, vias 0 -> 3
- net DATA_4_IN: track 166.9 -> 476.1 mm, vias 0 -> 3
- net DATA_OUT4: track 0.00 -> 302.7 mm, vias 0 -> 3
- net DATA_3_IN: track 169.6 -> 421.3 mm, vias 0 -> 3
- net DATA_OUT3: track 0.00 -> 247.4 mm, vias 0 -> 3
- net DATA_2_IN: track 167.5 -> 369.0 mm, vias 0 -> 3
- net DATA_OUT2: track 0.00 -> 193.2 mm, vias 0 -> 3
- net TR11: track 1408.8 -> 1577.9 mm, vias 17 -> 18
- net TR41: track 1467.6 -> 1636.1 mm, vias 18 -> 20
- net TR21: track 1862.7 -> 2026.8 mm, vias 162 -> 170
- net TR31: track 1830.6 -> 1993.1 mm, vias 158 -> 163
- net DATA_4: track 0.00 -> 157.3 mm, vias 0 -> 2
- net DATA_3: track 0.00 -> 156.5 mm, vias 0 -> 2
- net DATA_2: track 0.00 -> 156.2 mm, vias 0 -> 2
- net DATA_OUT1: track 0.00 -> 138.9 mm, vias 0 -> 3
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