File: P10_LED_2.kicad_pcb (KiCad board)
At the start: 2 copper layers, 711 parts, among them J1 2 Pin 5.5mm Male Molex OUTPUT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, J2 2 Pin 5.5mm Male Molex INPUT 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, J3 2 Pin 5.5mm Male Molex MAINS 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, J4 5 PIN 2.54MM PITCH BURGSTRIP, J5 5-PIN 2.54MM PITCH MALE STRAI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, J6 5-PIN 2.54MM PITCH MALE STRAI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, J7 Conn_02x07_Odd_Even, J8 Conn_02x07_Odd_Even, SW1 SW_DIP_x04, U1 STP16CPC26T, U10 STM32401VBT6 100 PIN LQFP, U11 MAX3483, U12 MX25L6406EM21, U2 STP16CPC26T, U3 STP16CPC26T, U4 STP16CPC26T, U5 STP16CPC26T, U6 STP16CPC26T, U7 STP16CPC26T, U8 STP16CPC26T, U9 MP24943DN-LF-Z SOIC8E

Commit message: update
Routing:
- net GND: track 1519.2 -> 2014.5 mm, vias 20 -> 34
- net TR41: track 1636.1 -> 1631.7 mm, vias 20 -> 21
- net TR11: vias 18 -> 20
- net TR31: track 1993.1 -> 1993.2 mm, vias 163 -> 165
- net TR21: vias 170 -> 172
